File: hardware/column_controller.brd (EAGLE design)
At the start: 160 x 100 mm, 35 parts, among them J4 JTAG, U1 ESP-WROVER-32ESP-WROVER-32, U2 3.3V, U3 CP2102N

Commit message: CAM
Parts:
- added FD1, FD2, FD3, FD4: FIDUCIAL1X2, SparkFun-Aesthetics:FIDUCIAL-1X2
- added H1, H2, H3, H4: STAND-OFF, SparkFun-Hardware:STAND-OFF
- added R10, R11: 5.1k, SparkFun-Resistors:0603
- moved J2 174.8 mm to (26.7, 1.27), turned to 180 degrees
- moved J1 173.9 mm to (25.4, 14.0)
- moved D4 171.9 mm to (12.4, 21.6), turned to 90 degrees
- moved R9 168.4 mm to (14.0, 21.6), turned to 90 degrees
- moved C11 158.1 mm to (32.4, 30.8)
- moved R8 153.9 mm to (17.1, 9.21), turned to 270 degrees
- moved C10 153.2 mm to (32.4, 29.2)
- moved R7 149.8 mm to (15.6, 9.21), turned to 90 degrees
- moved C9 148.3 mm to (32.4, 27.6)
- moved U3 145.8 mm to (11.4, 11.4), turned to 90 degrees
- moved R6 145.0 mm to (8.89, 16.5), turned to 90 degrees
- moved C8 143.2 mm to (28.6, 27.6), turned to 180 degrees
- moved R5 143.0 mm to (14.0, 16.5), turned to 270 degrees
- moved C7 141.2 mm to (28.6, 29.2), turned to 180 degrees
- moved C6 139.2 mm to (28.6, 30.8), turned to 180 degrees
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Connections:
- new net N$10: J3.A5, R11.2
- new net N$11: J3.B5, R10.2
- new net SHLD: J3.SHLD1, J3.SHLD2, J3.SHLD3, J3.SHLD4, J3.SHLD5, J3.SHLD6, J3.SHLD7, J3.SHLD8
- net 13: no longer R9.2
- net 3.3V: now also R9.2
- net GND: now also J3.GND, J3.GND2, R10.1, R11.1
Routing:
- net 3.3V: track 0.00 -> 108.3 mm, vias 0 -> 5
- net 5V: track 0.00 -> 57.7 mm
- net RX: track 0.00 -> 57.7 mm, vias 0 -> 2
- net TX: track 0.00 -> 57.3 mm
- net 0: track 0.00 -> 42.4 mm, vias 0 -> 2
- net !RESET: track 0.00 -> 41.2 mm, vias 0 -> 2
- net GND: track 0.00 -> 40.2 mm, vias 0 -> 42
- net VIN: track 0.00 -> 34.4 mm
- net V_USB: track 0.00 -> 31.9 mm, vias 0 -> 3
- net N$11: track 0.00 -> 24.8 mm
- net SCL: track 0.00 -> 19.5 mm
- net SDA: track 0.00 -> 19.2 mm
- net DTR: track 0.00 -> 17.8 mm, vias 0 -> 2
- net DOUT: track 0.00 -> 17.3 mm, vias 0 -> 2
- net N$3: track 0.00 -> 14.1 mm
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- added copper zone on layer 1, net GND
- added copper zone on layer 16, net GND
- added copper zone on layer 1, net SHLD
- added copper zone on layer 16, net SHLD
Other:
- board size 160 x 100 mm -> 35.6 x 54.6 mm
- board text added: "+"
- board text added: "-"
- board text added: "0"
- board text added: "RESET"
- board text added: "v02"
