File: hardware/2_sensor_board/color_sensor_node.sch (EAGLE design)
At the start: 19 parts, among them J1 JTAG, J2 JTAG, U1 ISL29125, U2 3.3V, U3 WS2811

Commit message: increase standoff size sensor board
Parts:
- H1, H2, H3, H4: value STAND-OFF -> STAND-OFF#8; device SparkFun-Hardware:STAND-OFF -> standoff:STAND-OFF#8
Changed lines of the file:
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@@
 <part name="GND8" library="SparkFun-PowerSymbols" deviceset="GND" device=""/>
 <part name="GND9" library="SparkFun-PowerSymbols" deviceset="GND" device=""/>
-<part name="H1" library="SparkFun-Hardware" deviceset="STAND-OFF" device=""/>
-<part name="H2" library="SparkFun-Hardware" deviceset="STAND-OFF" device=""/>
-<part name="H3" library="SparkFun-Hardware" deviceset="STAND-OFF" device=""/>
-<part name="H4" library="SparkFun-Hardware" deviceset="STAND-OFF" device=""/>
+<part name="H1" library="standoff" deviceset="STAND-OFF" device="#8"/>
+<part name="H2" library="standoff" deviceset="STAND-OFF" device="#8"/>
+<part name="H3" library="standoff" deviceset="STAND-OFF" device="#8"/>
+<part name="H4" library="standoff" deviceset="STAND-OFF" device="#8"/>
 <part name="FD1" library="SparkFun-Aesthetics" deviceset="FIDUCIAL" device="1X2" value="FIDUCIAL1X2"/>
 <part name="FD2" library="SparkFun-Aesthetics" deviceset="FIDUCIAL" device="1X2" value="FIDUCIAL1X2"/>

Commit message: prepare for v10 generation
Parts:
- FRAME1: DESIGNER (none) -> Owen Lyke; REV (none) -> v10
Changed lines of the file:
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@@
 <?xml version="1.0" encoding="utf-8"?>
 <!DOCTYPE eagle SYSTEM "eagle.dtd">
-<eagle version="9.6.0">
+<eagle version="9.2.0">
 <drawing>
 <settings>
@@
 </classes>
 <parts>
-<part name="FRAME1" library="SparkFun-Aesthetics" deviceset="FRAME-LETTER" device=""/>
+<part name="FRAME1" library="SparkFun-Aesthetics" deviceset="FRAME-LETTER" device="">
+<attribute name="DESIGNER" value="Owen Lyke"/>
+<attribute name="REV" value="v10"/>
+</part>
 <part name="U1" library="SparkFun-Sensors" deviceset="ISL29125" device=""/>
 <part name="U2" library="SparkFun-IC-Power" deviceset="V_REG_AP2112" device="K-3.3V" value="3.3V"/>
@@
 </plain>
 <instances>
-<instance part="FRAME1" gate="G$1" x="0" y="0" smashed="yes"/>
-<instance part="FRAME1" gate="V" x="147.32" y="0" smashed="yes">
+<instance part="FRAME1" gate="G$1" x="0" y="0"/>
+<instance part="FRAME1" gate="V" x="147.32" y="0">
 <attribute name="LAST_DATE_TIME" x="160.02" y="1.27" size="2.54" layer="94" font="vector"/>
 <attribute name="SHEET" x="233.68" y="1.27" size="2.54" layer="94" font="vector"/>
@@
 <attribute name="REV" x="236.22" y="6.604" size="2.7432" layer="94" font="vector"/>
 </instance>
-<instance part="U1" gate="G$1" x="71.12" y="83.82" smashed="yes">
+<instance part="U1" gate="G$1" x="71.12" y="83.82">
 <attribute name="NAME" x="63.5" y="89.154" size="1.778" layer="95" font="vector"/>
 <attribute name="VALUE" x="63.5" y="78.486" size="1.778" layer="96" font="vector" align="top-left"/>
 </instance>
-<instance part="U2" gate="G$1" x="198.12" y="137.16" smashed="yes">
+<instance part="U2" gate="G$1" x="198.12" y="137.16">
 <attribute name="NAME" x="190.5" y="145.034" size="1.778" layer="95" font="vector"/>
 <attribute name="VALUE" x="190.5" y="129.286" size="1.778" layer="96" font="vector" align="top-left"/>
 </instance>
-<instance part="SUPPLY1" gate="G$1" x="175.26" y="144.78" smashed="yes">
+<instance part="SUPPLY1" gate="G$1" x="175.26" y="144.78">
 <attribute name="VALUE" x="175.26" y="147.574" size="1.778" layer="96" align="bottom-center"/>
 </instance>
-<instance part="SUPPLY2" gate="G$1" x="210.82" y="144.78" smashed="yes">
+<instance part="SUPPLY2" gate="G$1" x="210.82" y="144.78">
 <attribute name="VALUE" x="210.82" y="147.574" size="1.778" layer="96" align="bottom-center"/>
 </instance>
-<instance part="C1" gate="G$1" x="175.26" y="134.62" smashed="yes">
+<instance part="C1" gate="G$1" x="175.26" y="134.62">
 <attribute name="NAME" x="176.784" y="137.541" size="1.778" layer="95" font="vector"/>
 <attribute name="VALUE" x="176.784" y="132.461" size="1.778" layer="96" font="vector"/>
 </instance>
-<instance part="GND1" gate="1" x="185.42" y="127" smashed="yes">
+<instance part="GND1" gate="1" x="185.42" y="127">
 <attribute name="VALUE" x="185.42" y="126.746" size="1.778" layer="96" align="top-center"/>
 </instance>
-<instance part="GND2" gate="1" x="210.82" y="127" smashed="yes">
+<instance part="GND2" gate="1" x="210.82" y="127">
 <attribute name="VALUE" x="210.82" y="126.746" size="1.778" layer="96" align="top-center"/>
 </instance>
-<instance part="GND3" gate="1" x="175.26" y="127" smashed="yes">
+<instance part="GND3" gate="1" x="175.26" y="127">
 <attribute name="VALUE" x="175.26" y="126.746" size="1.778" layer="96" align="top-center"/>
 </instance>
-<instance part="GND4" gate="1" x="48.26" y="76.2" smashed="yes">
+<instance part="GND4" gate="1" x="48.26" y="76.2">
 <attribute name="VALUE" x="48.26" y="75.946" size="1.778" layer="96" align="top-center"/>
 </instance>
-<instance part="C2" gate="G$1" x="210.82" y="134.62" smashed="yes">
+<instance part="C2" gate="G$1" x="210.82" y="134.62">
 <attribute name="NAME" x="212.344" y="137.541" size="1.778" layer="95" font="vector"/>
 <attribute name="VALUE" x="212.344" y="132.461" size="1.778" layer="96" font="vector"/>
 </instance>
-<instance part="D1" gate="G$1" x="73.66" y="134.62" smashed="yes">
+<instance part="D1" gate="G$1" x="73.66" y="134.62">
 <attribute name="NAME" x="71.12" y="143.002" size="1.778" layer="95" font="vector" align="bottom-center"/>
 </instance>
-<instance part="U3" gate="G$1" x="71.12" y="109.22" smashed="yes"/>
-<instance part="GND5" gate="1" x="55.88" y="101.6" smashed="yes">
+<instance part="U3" gate="G$1" x="71.12" y="109.22"/>
+<instance part="GND5" gate="1" x="55.88" y="101.6">
 <attribute name="VALUE" x="55.88" y="101.346" size="1.778" layer="96" align="top-center"/>
 </instance>
-<instance part="SUPPLY6" gate="G$1" x="53.34" y="142.24" smashed="yes">
+<instance part="SUPPLY6" gate="G$1" x="53.34" y="142.24">
 <attribute name="VALUE" x="53.34" y="145.034" size="1.778" layer="96" align="bottom-center"/>
 </instance>
-<instance part="GND6" gate="1" x="96.52" y="101.6" smashed="yes">
+<instance part="GND6" gate="1" x="96.52" y="101.6">
 <attribute name="VALUE" x="96.52" y="101.346" size="1.778" layer="96" align="top-center"/>
 </instance>
-<instance part="SUPPLY3" gate="G$1" x="48.26" y="142.24" smashed="yes">
+<instance part="SUPPLY3" gate="G$1" x="48.26" y="142.24">
 <attribute name="VALUE" x="48.26" y="145.034" size="1.778" layer="96" align="bottom-center"/>
 </instance>
-<instance part="R2" gate="G$1" x="48.26" y="129.54" smashed="yes" rot="R90">
+<instance part="R2" gate="G$1" x="48.26" y="129.54" rot="R90">
 <attribute name="NAME" x="46.736" y="129.54" size="1.778" layer="95" font="vector" rot="R90" align="bottom-center"/>
 <attribute name="VALUE" x="49.784" y="129.54" size="1.778" layer="96" font="vector" rot="R90" align="top-center"/>
 </instance>
-<instance part="SUPPLY8" gate="G$1" x="213.36" y="111.76" smashed="yes">
+<instance part="SUPPLY8" gate="G$1" x="213.36" y="111.76">
 <attribute name="VALUE" x="213.36" y="114.554" size="1.778" layer="96" align="bottom-center"/>
 </instance>
-<instance part="SUPPLY9" gate="G$1" x="213.36" y="86.36" smashed="yes">
+<instance part="SUPPLY9" gate="G$1" x="213.36" y="86.36">
 <attribute name="VALUE" x="213.36" y="89.154" size="1.778" layer="96" align="bottom-center"/>
 </instance>
-<instance part="GND8" gate="1" x="210.82" y="96.52" smashed="yes">
+<instance part="GND8" gate="1" x="210.82" y="96.52">
 <attribute name="VALUE" x="210.82" y="96.266" size="1.778" layer="96" align="top-center"/>
 </instance>
-<instance part="GND9" gate="1" x="210.82" y="71.12" smashed="yes">
+<instance part="GND9" gate="1" x="210.82" y="71.12">
 <attribute name="VALUE" x="210.82" y="70.866" size="1.778" layer="96" align="top-center"/>
 </instance>
-<instance part="H1" gate="G$1" x="223.52" y="33.02" smashed="yes"/>
-<instance part="H2" gate="G$1" x="226.06" y="33.02" smashed="yes"/>
-<instance part="H3" gate="G$1" x="226.06" y="30.48" smashed="yes"/>
-<instance part="H4" gate="G$1" x="223.52" y="30.48" smashed="yes"/>
-<instance part="FD1" gate="G$1" x="231.14" y="33.02" smashed="yes"/>
-<instance part="FD2" gate="G$1" x="231.14" y="30.48" smashed="yes"/>
-<instance part="FD3" gate="G$1" x="233.68" y="30.48" smashed="yes"/>
-<instance part="FD4" gate="G$1" x="233.68" y="33.02" smashed="yes"/>
-<instance part="GND7" gate="1" x="175.26" y="96.52" smashed="yes">
+<instance part="H1" gate="G$1" x="223.52" y="33.02"/>
+<instance part="H2" gate="G$1" x="226.06" y="33.02"/>
+<instance part="H3" gate="G$1" x="226.06" y="30.48"/>
+<instance part="H4" gate="G$1" x="223.52" y="30.48"/>
+<instance part="FD1" gate="G$1" x="231.14" y="33.02"/>
+<instance part="FD2" gate="G$1" x="231.14" y="30.48"/>
+<instance part="FD3" gate="G$1" x="233.68" y="30.48"/>
+<instance part="FD4" gate="G$1" x="233.68" y="33.02"/>
+<instance part="GND7" gate="1" x="175.26" y="96.52">
 <attribute name="VALUE" x="175.26" y="96.266" size="1.778" layer="96" align="top-center"/>
 </instance>
-<instance part="SUPPLY7" gate="G$1" x="172.72" y="111.76" smashed="yes">
+<instance part="SUPPLY7" gate="G$1" x="172.72" y="111.76">
 <attribute name="VALUE" x="172.72" y="114.554" size="1.778" layer="96" align="bottom-center"/>
 </instance>
-<instance part="GND10" gate="1" x="175.26" y="71.12" smashed="yes">
+<instance part="GND10" gate="1" x="175.26" y="71.12">
 <attribute name="VALUE" x="175.26" y="70.866" size="1.778" layer="96" align="top-center"/>
 </instance>
-<instance part="SUPPLY10" gate="G$1" x="172.72" y="86.36" smashed="yes">
+<instance part="SUPPLY10" gate="G$1" x="172.72" y="86.36">
 <attribute name="VALUE" x="172.72" y="89.154" size="1.778" layer="96" align="bottom-center"/>
 </instance>
-<instance part="J1" gate="J1" x="193.04" y="106.68" smashed="yes">
+<instance part="J1" gate="J1" x="193.04" y="106.68">
 <attribute name="NAME" x="180.34" y="114.554" size="1.778" layer="95" font="vector"/>
 <attribute name="VALUE" x="180.34" y="96.774" size="1.778" layer="96" font="vector"/>
 </instance>
-<instance part="J2" gate="J1" x="193.04" y="81.28" smashed="yes">
+<instance part="J2" gate="J1" x="193.04" y="81.28">
 <attribute name="NAME" x="180.34" y="89.154" size="1.778" layer="95" font="vector"/>
 <attribute name="VALUE" x="180.34" y="71.374" size="1.778" layer="96" font="vector"/>
 </instance>
-<instance part="C3" gate="G$1" x="48.26" y="86.36" smashed="yes">
+<instance part="C3" gate="G$1" x="48.26" y="86.36">
 <attribute name="NAME" x="49.784" y="89.281" size="1.778" layer="95" font="vector"/>
 <attribute name="VALUE" x="49.784" y="84.201" size="1.778" layer="96" font="vector"/>
