File: hardware/1_backer_board/sensor_node_backer.brd (EAGLE design)
At the start: 27.9 x 30.5 mm, 8 parts

Commit message: increase standoff size backer
Parts:
- H1, H2, H3, H4: device SparkFun-Hardware:STAND-OFF -> standoff:STAND-OFF-#8
Other:
- board text added: "v03"
- board text removed: "v02"
Changed lines of the file:
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@@
 <wire x1="25.25666875" y1="30.48" x2="2.54" y2="30.48" width="0" layer="20"/>
 <wire x1="2.54" y1="30.48" x2="0.00909375" y2="27.9479375" width="0" layer="20" curve="90.026176"/>
-<text x="10.668" y="0.381" size="1.778" layer="16" font="vector" ratio="15" rot="SMR0">v02</text>
+<text x="10.668" y="0.381" size="1.778" layer="16" font="vector" ratio="15" rot="SMR0">v03</text>
 <rectangle x1="10.795" y1="19.05" x2="17.145" y2="28.575" layer="51"/>
 <hole x="10.795" y="28.575" drill="1.27"/>
@@
 </autorouter>
 <elements>
-<element name="H1" library="SparkFun-Hardware" package="STAND-OFF" value="STAND-OFF" x="25.4" y="2.54" smashed="yes">
+<element name="H1" library="standoff" package="STAND-OFF-#8" value="STAND-OFF" x="25.4" y="2.54" smashed="yes">
 <attribute name="NAME" x="25.4" y="4.572" size="0.6096" layer="25" font="vector" ratio="20" align="bottom-center"/>
 <attribute name="VALUE" x="25.4" y="0.508" size="0.6096" layer="27" font="vector" ratio="20" align="top-center"/>
 </element>
-<element name="H2" library="SparkFun-Hardware" package="STAND-OFF" value="STAND-OFF" x="2.54" y="2.54" smashed="yes">
+<element name="H2" library="standoff" package="STAND-OFF-#8" value="STAND-OFF" x="2.54" y="2.54" smashed="yes">
 <attribute name="NAME" x="2.54" y="4.572" size="0.6096" layer="25" font="vector" ratio="20" align="bottom-center"/>
 <attribute name="VALUE" x="2.54" y="0.508" size="0.6096" layer="27" font="vector" ratio="20" align="top-center"/>
 </element>
-<element name="H3" library="SparkFun-Hardware" package="STAND-OFF" value="STAND-OFF" x="25.4" y="27.94" smashed="yes">
+<element name="H3" library="standoff" package="STAND-OFF-#8" value="STAND-OFF" x="25.4" y="27.94" smashed="yes">
 <attribute name="NAME" x="25.4" y="29.972" size="0.6096" layer="25" font="vector" ratio="20" align="bottom-center"/>
 <attribute name="VALUE" x="25.4" y="25.908" size="0.6096" layer="27" font="vector" ratio="20" align="top-center"/>
 </element>
-<element name="H4" library="SparkFun-Hardware" package="STAND-OFF" value="STAND-OFF" x="2.54" y="27.94" smashed="yes">
+<element name="H4" library="standoff" package="STAND-OFF-#8" value="STAND-OFF" x="2.54" y="27.94" smashed="yes">
 <attribute name="NAME" x="2.54" y="29.972" size="0.6096" layer="25" font="vector" ratio="20" align="bottom-center"/>
 <attribute name="VALUE" x="2.54" y="25.908" size="0.6096" layer="27" font="vector" ratio="20" align="top-center"/>

Commit message: prepare for v10 generation
Other:
- board text added: "v10"
- board text removed: "v03"
Changed lines of the file:
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@@
 <?xml version="1.0" encoding="utf-8"?>
 <!DOCTYPE eagle SYSTEM "eagle.dtd">
-<eagle version="9.6.0">
+<eagle version="9.2.0">
 <drawing>
 <settings>
@@
 <setting verticaltext="up"/>
 </settings>
-<grid distance="50" unitdist="mil" unit="mil" style="lines" multiple="1" display="yes" altdistance="5" altunitdist="mil" altunit="mil"/>
+<grid distance="0.05" unitdist="inch" unit="inch" style="lines" multiple="1" display="yes" altdistance="0.005" altunitdist="inch" altunit="inch"/>
 <layers>
 <layer number="1" name="Top" color="4" fill="1" visible="yes" active="yes"/>
@@
 <wire x1="25.25666875" y1="30.48" x2="2.54" y2="30.48" width="0" layer="20"/>
 <wire x1="2.54" y1="30.48" x2="0.00909375" y2="27.9479375" width="0" layer="20" curve="90.026176"/>
-<text x="10.668" y="0.381" size="1.778" layer="16" font="vector" ratio="15" rot="SMR0">v03</text>
+<text x="10.668" y="0.381" size="1.778" layer="16" font="vector" ratio="15" rot="SMR0">v10</text>
 <rectangle x1="10.795" y1="19.05" x2="17.145" y2="28.575" layer="51"/>
 <hole x="10.795" y="28.575" drill="1.27"/>
@@
 </autorouter>
 <elements>
-<element name="H1" library="standoff" package="STAND-OFF-#8" value="STAND-OFF" x="25.4" y="2.54" smashed="yes">
+<element name="H1" library="standoff" package="STAND-OFF-#8" value="STAND-OFF" x="25.4" y="2.54">
 <attribute name="NAME" x="25.4" y="4.572" size="0.6096" layer="25" font="vector" ratio="20" align="bottom-center"/>
 <attribute name="VALUE" x="25.4" y="0.508" size="0.6096" layer="27" font="vector" ratio="20" align="top-center"/>
 </element>
-<element name="H2" library="standoff" package="STAND-OFF-#8" value="STAND-OFF" x="2.54" y="2.54" smashed="yes">
+<element name="H2" library="standoff" package="STAND-OFF-#8" value="STAND-OFF" x="2.54" y="2.54">
 <attribute name="NAME" x="2.54" y="4.572" size="0.6096" layer="25" font="vector" ratio="20" align="bottom-center"/>
 <attribute name="VALUE" x="2.54" y="0.508" size="0.6096" layer="27" font="vector" ratio="20" align="top-center"/>
 </element>
-<element name="H3" library="standoff" package="STAND-OFF-#8" value="STAND-OFF" x="25.4" y="27.94" smashed="yes">
+<element name="H3" library="standoff" package="STAND-OFF-#8" value="STAND-OFF" x="25.4" y="27.94">
 <attribute name="NAME" x="25.4" y="29.972" size="0.6096" layer="25" font="vector" ratio="20" align="bottom-center"/>
 <attribute name="VALUE" x="25.4" y="25.908" size="0.6096" layer="27" font="vector" ratio="20" align="top-center"/>
 </element>
-<element name="H4" library="standoff" package="STAND-OFF-#8" value="STAND-OFF" x="2.54" y="27.94" smashed="yes">
+<element name="H4" library="standoff" package="STAND-OFF-#8" value="STAND-OFF" x="2.54" y="27.94">
 <attribute name="NAME" x="2.54" y="29.972" size="0.6096" layer="25" font="vector" ratio="20" align="bottom-center"/>
 <attribute name="VALUE" x="2.54" y="25.908" size="0.6096" layer="27" font="vector" ratio="20" align="top-center"/>
 </element>
-<element name="FD1" library="SparkFun-Aesthetics" package="FIDUCIAL-1X2" value="FIDUCIAL1X2" x="5.08" y="25.4" smashed="yes"/>
-<element name="FD2" library="SparkFun-Aesthetics" package="FIDUCIAL-1X2" value="FIDUCIAL1X2" x="22.86" y="5.08" smashed="yes"/>
-<element name="FD3" library="SparkFun-Aesthetics" package="FIDUCIAL-1X2" value="FIDUCIAL1X2" x="5.08" y="25.4" smashed="yes" rot="MR0"/>
-<element name="FD4" library="SparkFun-Aesthetics" package="FIDUCIAL-1X2" value="FIDUCIAL1X2" x="22.86" y="5.08" smashed="yes" rot="MR0"/>
+<element name="FD1" library="SparkFun-Aesthetics" package="FIDUCIAL-1X2" value="FIDUCIAL1X2" x="5.08" y="25.4"/>
+<element name="FD2" library="SparkFun-Aesthetics" package="FIDUCIAL-1X2" value="FIDUCIAL1X2" x="22.86" y="5.08"/>
+<element name="FD3" library="SparkFun-Aesthetics" package="FIDUCIAL-1X2" value="FIDUCIAL1X2" x="5.08" y="25.4" rot="MR0"/>
+<element name="FD4" library="SparkFun-Aesthetics" package="FIDUCIAL-1X2" value="FIDUCIAL1X2" x="22.86" y="5.08" rot="MR0"/>
 </elements>
 <signals>

Commit message: v10 CAM + Gerber Gen
Other:
- board text added: "ROUTE OUT"
Changed lines of the file:
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@@
 <?xml version="1.0" encoding="utf-8"?>
 <!DOCTYPE eagle SYSTEM "eagle.dtd">
-<eagle version="9.2.0">
+<eagle version="9.6.0">
 <drawing>
 <settings>
@@
 <setting verticaltext="up"/>
 </settings>
-<grid distance="0.05" unitdist="inch" unit="inch" style="lines" multiple="1" display="yes" altdistance="0.005" altunitdist="inch" altunit="inch"/>
+<grid distance="50" unitdist="mil" unit="mil" style="lines" multiple="1" display="yes" altdistance="5" altunitdist="mil" altunit="mil"/>
 <layers>
 <layer number="1" name="Top" color="4" fill="1" visible="yes" active="yes"/>
@@
 <circle x="13.97" y="9.525" radius="7.62" width="0.0254" layer="20"/>
 <text x="23.749" y="0.254" size="1.778" layer="16" font="vector" ratio="15" rot="MR0">BACKER</text>
+<text x="13.97" y="20.32" size="1.016" layer="1" font="vector" ratio="15" rot="R90">ROUTE OUT</text>
+<text x="10.16" y="8.89" size="1.016" layer="1" font="vector" ratio="15">ROUTE OUT</text>
 </plain>
 <attributes>
@@
 </autorouter>
 <elements>
-<element name="H1" library="standoff" package="STAND-OFF-#8" value="STAND-OFF" x="25.4" y="2.54">
+<element name="H1" library="standoff" package="STAND-OFF-#8" value="STAND-OFF" x="25.4" y="2.54" smashed="yes">
 <attribute name="NAME" x="25.4" y="4.572" size="0.6096" layer="25" font="vector" ratio="20" align="bottom-center"/>
 <attribute name="VALUE" x="25.4" y="0.508" size="0.6096" layer="27" font="vector" ratio="20" align="top-center"/>
 </element>
-<element name="H2" library="standoff" package="STAND-OFF-#8" value="STAND-OFF" x="2.54" y="2.54">
+<element name="H2" library="standoff" package="STAND-OFF-#8" value="STAND-OFF" x="2.54" y="2.54" smashed="yes">
 <attribute name="NAME" x="2.54" y="4.572" size="0.6096" layer="25" font="vector" ratio="20" align="bottom-center"/>
 <attribute name="VALUE" x="2.54" y="0.508" size="0.6096" layer="27" font="vector" ratio="20" align="top-center"/>
 </element>
-<element name="H3" library="standoff" package="STAND-OFF-#8" value="STAND-OFF" x="25.4" y="27.94">
+<element name="H3" library="standoff" package="STAND-OFF-#8" value="STAND-OFF" x="25.4" y="27.94" smashed="yes">
 <attribute name="NAME" x="25.4" y="29.972" size="0.6096" layer="25" font="vector" ratio="20" align="bottom-center"/>
 <attribute name="VALUE" x="25.4" y="25.908" size="0.6096" layer="27" font="vector" ratio="20" align="top-center"/>
 </element>
-<element name="H4" library="standoff" package="STAND-OFF-#8" value="STAND-OFF" x="2.54" y="27.94">
+<element name="H4" library="standoff" package="STAND-OFF-#8" value="STAND-OFF" x="2.54" y="27.94" smashed="yes">
 <attribute name="NAME" x="2.54" y="29.972" size="0.6096" layer="25" font="vector" ratio="20" align="bottom-center"/>
 <attribute name="VALUE" x="2.54" y="25.908" size="0.6096" layer="27" font="vector" ratio="20" align="top-center"/>
 </element>
-<element name="FD1" library="SparkFun-Aesthetics" package="FIDUCIAL-1X2" value="FIDUCIAL1X2" x="5.08" y="25.4"/>
-<element name="FD2" library="SparkFun-Aesthetics" package="FIDUCIAL-1X2" value="FIDUCIAL1X2" x="22.86" y="5.08"/>
-<element name="FD3" library="SparkFun-Aesthetics" package="FIDUCIAL-1X2" value="FIDUCIAL1X2" x="5.08" y="25.4" rot="MR0"/>
-<element name="FD4" library="SparkFun-Aesthetics" package="FIDUCIAL-1X2" value="FIDUCIAL1X2" x="22.86" y="5.08" rot="MR0"/>
+<element name="FD1" library="SparkFun-Aesthetics" package="FIDUCIAL-1X2" value="FIDUCIAL1X2" x="5.08" y="25.4" smashed="yes"/>
+<element name="FD2" library="SparkFun-Aesthetics" package="FIDUCIAL-1X2" value="FIDUCIAL1X2" x="22.86" y="5.08" smashed="yes"/>
+<element name="FD3" library="SparkFun-Aesthetics" package="FIDUCIAL-1X2" value="FIDUCIAL1X2" x="5.08" y="25.4" smashed="yes" rot="MR0"/>
+<element name="FD4" library="SparkFun-Aesthetics" package="FIDUCIAL-1X2" value="FIDUCIAL1X2" x="22.86" y="5.08" smashed="yes" rot="MR0"/>
 </elements>
 <signals>
